Commit message: refactor

File: teleop/urdf/robot_fixed.urdf (robot description, URDF)
Before this commit: robot opus, 18 links, 17 joints
Joints:
- joint left_elbow_yaw: type fixed -> revolute
- joint left_shoulder_pitch: type fixed -> revolute
- joint left_shoulder_yaw: type fixed -> revolute
- joint right_elbow_yaw: type fixed -> revolute
- joint right_shoulder_pitch: type fixed -> revolute
- joint right_shoulder_yaw: type fixed -> revolute
